File: DAC.kicad_sch (KiCad schematic)
At the start: 43 parts, among them J2 PJ-3270, U10 OPA1652, U11 LM4562, U9 WM8741

Commit message: added winstar display
Parts:
- C26, C28, C30, C32, C33, C34, C37, C38, C45, C46: footprint (none) -> rlib_passive:C_0603_1608Metric
Changed lines of the file:
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@@
       (effects (font (size 1.27 1.27)) (justify left))
     )
-    (property "Footprint" "" (id 2) (at 144.4752 95.25 0)
+    (property "Footprint" "rlib_passive:C_0603_1608Metric" (id 2) (at 144.4752 95.25 0)
       (effects (font (size 1.27 1.27)) hide)
     )
@@
       (effects (font (size 1.27 1.27)) (justify left))
     )
-    (property "Footprint" "" (id 2) (at 101.2952 96.52 0)
+    (property "Footprint" "rlib_passive:C_0603_1608Metric" (id 2) (at 101.2952 96.52 0)
       (effects (font (size 1.27 1.27)) hide)
     )
@@
       (effects (font (size 1.27 1.27)) (justify left))
     )
-    (property "Footprint" "" (id 2) (at 158.4452 130.81 0)
+    (property "Footprint" "rlib_passive:C_0603_1608Metric" (id 2) (at 158.4452 130.81 0)
       (effects (font (size 1.27 1.27)) hide)
     )
@@
       (effects (font (size 1.27 1.27)) (justify left))
     )
-    (property "Footprint" "" (id 2) (at 86.0552 96.52 0)
+    (property "Footprint" "rlib_passive:C_0603_1608Metric" (id 2) (at 86.0552 96.52 0)
       (effects (font (size 1.27 1.27)) hide)
     )
@@
       (effects (font (size 1.27 1.27)) (justify left))
     )
-    (property "Footprint" "" (id 2) (at 213.0552 129.54 0)
+    (property "Footprint" "rlib_passive:C_0603_1608Metric" (id 2) (at 213.0552 129.54 0)
       (effects (font (size 1.27 1.27)) hide)
     )
@@
       (effects (font (size 1.27 1.27)) (justify left))
     )
-    (property "Footprint" "" (id 2) (at 143.2052 48.26 0)
+    (property "Footprint" "rlib_passive:C_0603_1608Metric" (id 2) (at 143.2052 48.26 0)
       (effects (font (size 1.27 1.27)) hide)
     )
@@
       (effects (font (size 1.27 1.27)) (justify left))
     )
-    (property "Footprint" "" (id 2) (at 158.4452 143.51 0)
+    (property "Footprint" "rlib_passive:C_0603_1608Metric" (id 2) (at 158.4452 143.51 0)
       (effects (font (size 1.27 1.27)) hide)
     )
@@
       (effects (font (size 1.27 1.27)) (justify left))
     )
-    (property "Footprint" "" (id 2) (at 92.4052 111.76 0)
+    (property "Footprint" "rlib_passive:C_0603_1608Metric" (id 2) (at 92.4052 111.76 0)
       (effects (font (size 1.27 1.27)) hide)
     )
@@
       (effects (font (size 1.27 1.27)) (justify left))
     )
-    (property "Footprint" "" (id 2) (at 213.0552 142.24 0)
+    (property "Footprint" "rlib_passive:C_0603_1608Metric" (id 2) (at 213.0552 142.24 0)
       (effects (font (size 1.27 1.27)) hide)
     )
@@
       (effects (font (size 1.27 1.27)) (justify left))
     )
-    (property "Footprint" "" (id 2) (at 116.5352 96.52 0)
-      (effects (font (size 1.27 1.27)) hide)
-    )
+    (property "Footprint" "rlib_passive:C_0603_1608Metric" (id 2) (at 116.5352 96.52 0)
+      (effects (font (size 1.27 1.27)) hide)
+    )
