File: SOC.kicad_sch (KiCad schematic)
At the start: 66 parts, among them J3 TF01-A, P1 HRO-TYPE-C-31-M-12, P2 WF24HTLAJDNN0#, Q1 Q_NMOS_DSG, SW2 TS-1157-X-A, SW3 TS-1157-X-A, SW4 TS-1157-X-A, SW5 TS-1157-X-A, SW6 TS-1157-X-A, SW7 TS-1010-C-A, SW8 TS-1010-C-A, U12 W25Q128JVSIQ, U4 F1C200S, U8 USBLC6-2SC6, Y1 Crystal_GND24

Commit message: added winstar display
Parts:
- added F2: Fuse, symbol Device:Fuse
- C15, C47, C48, C49, C50, C54, C55, C56, C57, C58, C59, C60, C61, C62, C63, C64, C65, C66, C67, C68, C69, C70, C71, C74, C75: footprint (none) -> rlib_passive:C_0603_1608Metric
Connections:
- net at P1.A4 (VBUS), P1.A9 (VBUS), P1.B4 (VBUS)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: now also F2.2; no longer C71.1, L9.2
- new net: C71.1, F2.1, L9.2
Other:
- note added: "LCD"
- moved on the sheet: C15, C60, C66, C67, C70, C71, J3, JP1, L9, P2, Q1, R29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

Commit message: buttons are changed
Parts:
- SW2: renamed from SW3; value TS-1157-X-A -> TS-1157-X-F; footprint rlib_buttons:TS-1157-X-A -> rlib_buttons:TS-1157-X-F; symbol rlib_buttons:TS-1157-X-A -> rlib_buttons:TS-1157-X-F
- SW3: renamed from SW6; value TS-1157-X-A -> TS-1157-X-F; footprint rlib_buttons:TS-1157-X-A -> rlib_buttons:TS-1157-X-F; symbol rlib_buttons:TS-1157-X-A -> rlib_buttons:TS-1157-X-F
- SW4, SW5: value TS-1157-X-A -> TS-1157-X-F; footprint rlib_buttons:TS-1157-X-A -> rlib_buttons:TS-1157-X-F; symbol rlib_buttons:TS-1157-X-A -> rlib_buttons:TS-1157-X-F
- SW6: renamed from SW2; value TS-1157-X-A -> TS-1157-X-F; footprint rlib_buttons:TS-1157-X-A -> rlib_buttons:TS-1157-X-F; symbol rlib_buttons:TS-1157-X-A -> rlib_buttons:TS-1157-X-F
Other:
- moved on the sheet: C66, J3, R34, R35, R36, R37
