File: hardware/SOC.kicad_sch (KiCad schematic)
At the start: 81 parts, among them J3 TF01-A, P1 HRO-TYPE-C-31-M-12, P2 WF24HTLAJDNN0#, Q1 Q_NMOS_DSG, SW2 K2-1156SP-F5SW-05, SW3 K2-1156SP-F5SW-05, SW4 K2-1156SP-F5SW-05, SW5 K2-1156SP-F5SW-05, SW6 K2-1156SP-F5SW-05, SW7 TS-1010-C-A, SW8 TS-1010-C-A, U12 MX25L25635F, U4 F1C200S, U8 USBLC6-2SC6, Y1 Crystal_GND24

Commit message: some changes
Parts:
- removed C49, C50, C69: 100n, rlib_passive:C_0603_1608Metric, symbol rlib_passive:C
- removed JP1: SolderJumper_3_Open, symbol Jumper:SolderJumper_3_Open
- removed P2: WF24HTLAJDNN0#, symbol rlib_lcd:WF24HTLAJDNN0#
- removed R41: R, rlib_passive:R_0603_1608Metric, symbol rlib_passive:R
- removed Y1: Crystal_GND24, rlib_crystals:Crystal_SMD_Abracon_ABM8G-4Pin_3.2x2.5mm, symbol rlib_crystal:Crystal_GND24
- added P2: WF24LTYAJDNN0#, rlib_lcd:WF24LTYAJDNN0, symbol rlib_lcd:WF24LTYAJDNN0#
- added R11, R12: 10k, rlib_passive:R_0603_1608Metric, symbol rlib_passive:R
- added TP17, TP18, TP19, TP6, TP8: TestPoint, symbol Connector:TestPoint
- added Y1: XRCGB24M000F1H01R0, rlib_crystals:OSC_XRCGB24M000F1H01R0, symbol rlib_crystal:XRCGB24M000F1H01R0
- F2: value Fuse -> 500mA; footprint (none) -> rlib_passive:FUSC3216X85N; symbol Device:Fuse -> rlib_passive:Fuse
- L9: footprint (none) -> rlib_passive:INDC2520X120N
- R34, R35, R36, R37, R39, R46, R47: value R -> 10k
- R38, R40: value R -> 100
- R43, R44: value R -> 27
- SW7, SW8: value TS-1010-C-A -> GT-TC054A-H035-L1
Connections:
- net +3V3: now also P2.36 (LEDK), P2.37 (LEDK), P2.7 (VCI), P2.8 (IOVCC), R11.2, R12.2
- net GND: now also P2.1 (GND), P2.31 (IM0), P2.32 (IM1), P2.33 (IM2); no longer C55.2, C58.2
- net KEYS: now also TP6.1
- net LCD_CS: now also P2.10 (CS), TP8.1
- net LCD_D0: now also P2.14 (DB0)
- net LCD_D1: now also P2.15 (DB1)
- net LCD_D10: now also P2.24 (DB10)
- net LCD_D11: now also P2.25 (DB11)
- net LCD_D12: now also P2.26 (DB12)
- net LCD_D13: now also P2.27 (DB13)
- net LCD_D14: now also P2.28 (DB14)
- net LCD_D15: now also P2.29 (DB15)
- net LCD_D2: now also P2.16 (DB2)
- net LCD_D3: now also P2.17 (DB3)
- net LCD_D4: now also P2.18 (DB4)
- net LCD_D5: now also P2.19 (DB5)
- net LCD_D6: now also P2.20 (DB6)
- net LCD_D7: now also P2.21 (DB7)
- net LCD_D8: now also P2.22 (DB8)
- net LCD_D9: now also P2.23 (DB9)
- net LCD_RD: now also P2.13 (RD), TP19.1
- net LCD_RS: now also P2.11 (D/CX), TP17.1
- net LCD_WR: now also P2.12 (WR), TP18.1
- net at C73.1, U4.51 (HOSCI): now also Y1.1
- net at C72.1, U4.52 (HOSCO): now also Y1.3
- net at R38.1: now also P2.38 (LEDA)
- net RESET: now reaches JP2.2 (B), U4.70 (RESET)
- net SD_PLUG: now reaches U4.40 (PE9/CSI_D6/UART2_RTS/SPI1_CLK/EINTE9)
- net SD_PLUG: now also J3.9 (CD), R12.1
- net HP_PLUG: no longer names the net of U4.42 (PE7/CSI_D4/UART2_TX/SPI1_CS/EINTE7)
- new net: P2.30 (RESET), R11.1
- new net: C55.2, C58.2
Other:
- moved on the sheet: C15, C47, C48, C60, C67, C70, C71, C72, C73, C74, C75, D4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
