File: new_hardware/_autosave-SOC.kicad_sch (KiCad schematic)
At the start: 88 parts, among them J3 TF01-A, P1 USB-TYPE-C-018, P2 WF24LTYAJDNN0#, Q1 Q_NMOS_DSG, SW2 K2-1156SP-F5SW-05, SW3 K2-1156SP-F5SW-05, SW4 K2-1156SP-F5SW-05, SW5 K2-1156SP-F5SW-05, SW6 K2-1156SP-F5SW-05, SW7 GT-TC054A-H035-L1, SW8 GT-TC054A-H035-L1, U2 F133, U8 USBLC6-2SC6, U9 MX25L25645GM2I-08G, Y1 12.88727

Commit message: some changes
Parts:
- gave numbers to parts that had none: 3
Changed lines of the file:
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@@
   (symbol (lib_id "rlib_passive:PESD3V3L1BA") (at 346.71 87.63 90) (unit 1)
     (in_bom yes) (on_board yes)
-    (property "Reference" "D?" (id 0) (at 343.9003 83.5772 90)
+    (property "Reference" "D3" (id 0) (at 343.9003 83.5772 90)
       (effects (font (size 1.27 1.27)) (justify right))
     )
@@
   (symbol (lib_id "Connector:TestPoint") (at 369.57 146.05 270) (unit 1)
     (in_bom yes) (on_board yes)
-    (property "Reference" "TP?" (id 0) (at 367.03 151.13 90)
+    (property "Reference" "TP15" (id 0) (at 367.03 151.13 90)
       (effects (font (size 1.27 1.27)) (justify left))
     )
@@
   (symbol (lib_id "Connector:TestPoint") (at 309.88 147.32 90) (unit 1)
     (in_bom yes) (on_board yes)
-    (property "Reference" "TP?" (id 0) (at 312.42 142.24 90)
-      (effects (font (size 1.27 1.27)) (justify left))
-    )
+    (property "Reference" "TP14" (id 0) (at 312.42 142.24 90)
+      (effects (font (size 1.27 1.27)) (justify left))
+    )
