File: new_hardware/mp3_test_board.kicad_pcb (KiCad board)
At the start: 4 copper layers, 100 x 56 mm, 210 parts, among them J1 TF01-A, J2 PJ-322, P1 WF24LTYAJDNN0#, P2 USB-TYPE-C-018, Q1 2N7002K, SW1 K2-1156SP-F5SW-05, SW2 K2-1156SP-F5SW-05, SW3 K2-1156SP-F5SW-05, SW4 K2-1156SP-F5SW-05, SW5 K2-1156SP-F5SW-05, SW6 GT-TC054A-H035-L1, SW7 GT-TC054A-H035-L1, SW8 GT-TC054A-H035-L1, U1 F133, U10 SGM6603-ADJYN6G, U11 SGM3204, U2 USBLC6-2SC6, U3 MX25L25645GM2I-08G, U4 PCM1795, U5 LM4562, U6 LM4562, U7 OPA1656, U8 OPA1656, U9 AXP2101, Y1 12.88727

Commit message: xxx
Parts:
- added R58: 10k, rlib_passive:R_0603_1608Metric, B.Cu at (111.1, 96.4)
- added R59: 10k, rlib_passive:R_0603_1608Metric, B.Cu at (111.1, 94.9)
- added R60: 10k, rlib_passive:R_0603_1608Metric, B.Cu at (111.1, 93.5)
- added R61: 10k, rlib_passive:R_0603_1608Metric, B.Cu at (111.1, 91.9)
- added R62: 10k, rlib_passive:R_0603_1608Metric, B.Cu at (111.1, 90.4)
- added R63: 10k, rlib_passive:R_0603_1608Metric, B.Cu at (130.2, 87.2)
- added R64: 10k, rlib_passive:R_0603_1608Metric, B.Cu at (106.7, 94.2)
- added R65: 10k, rlib_passive:R_0603_1608Metric, B.Cu at (111.1, 88.9)
- added RF1: BWIPX-1-001E, rlib_connectors:IPEX-SMD_BWIPX-1-001E, B.Cu at (104.0, 96.5)
- C56, C59, C60, C66, L1: moved to B.Cu
- moved U 72.3 mm to (121.8, 90.8), turned to 90 degrees
- moved C60 25.0 mm to (111.2, 85.3), turned to 180 degrees
- moved C66 24.5 mm to (111.2, 86.8), turned to 180 degrees
- moved C56 23.5 mm to (131.7, 97.5), turned to 90 degrees
- moved L1 20.6 mm to (106.9, 87.5), turned to 90 degrees
- moved C59 18.6 mm to (129.8, 97.5), turned to 90 degrees
- moved TP4 14.9 mm to (116.1, 73.6)
- moved TP21 14.3 mm to (139.3, 97.8)
- moved TP3 13.1 mm to (116.0, 75.7)
- moved TP2 11.8 mm to (116.1, 77.9)
- moved TP1 11.3 mm to (116.2, 80.0)
- moved TP22 11.1 mm to (135.7, 85.2)
- moved R7 10.5 mm to (93.9, 94.1)
- moved TP23 9.46 mm to (133.6, 86.5)
- moved R46 9.21 mm to (174.2, 70.2), turned to -90 degrees
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Connections:
- C60 pad 1: +3V3 -> Net-(C60-Pad1)
- L1 pad 2: +3V3 -> Net-(C60-Pad1)
- U pad 12: unconnected-(U12-Pad12) -> /WI-FI/WIFI_REG_ON
- U pad 2: unconnected-(U12-Pad2) -> Net-(U12-Pad2)
- U pad 23: +3V3 -> Net-(C60-Pad1)
- U pad 34: unconnected-(U12-Pad34) -> Net-(R63-Pad1)
Routing:
- net /Power/AUDIO_PWR_EN: track 18.1 -> 133.6 mm, vias 1 -> 2
- net /SOC/WIFI_SDIO_D2: track 2.86 -> 69.2 mm, vias 1 -> 2
- net /SOC/WIFI_SDIO_D3: track 2.68 -> 68.8 mm, vias 1 -> 2
- net +3V3: track 350.5 -> 413.1 mm, vias 20 -> 26
- net /SOC/WIFI_SDIO_D0: track 3.02 -> 64.9 mm, vias 1 -> 2
- net /SOC/WIFI_SDIO_D1: track 3.04 -> 64.3 mm, vias 1 -> 2
- net /SOC/WIFI_SDIO_CLK: track 3.67 -> 64.6 mm, vias 1 -> 2
- net /SOC/WIFI_SDIO_CMD: track 2.40 -> 61.7 mm, vias 1 -> 2
- net Net-(U12-Pad2): track 0.00 -> 26.1 mm, vias 0 -> 2
- net GND: track 312.5 -> 336.7 mm, vias 106 -> 130
- net Net-(D12-Pad1): track 98.0 -> 115.0 mm
- net /WI-FI/WIFI_REG_ON: track 0.00 -> 16.5 mm
- net /NewDAC/I2C_SCL: track 130.0 -> 146.1 mm
- net /NewDAC/I2C_SDIN: track 129.6 -> 145.5 mm
- net Net-(R10-Pad1): track 26.6 -> 11.6 mm, vias 2 -> 1
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- added copper zone on B.Cu, net +5VA
- added copper zone on B.Cu, net -5VA
- added copper zone on B.Cu, net Net-(C61-Pad1)
- added copper zone on B.Cu, net VBUS
- added copper zone on B.Cu, net VCC

Commit message: removed some dirs
Routing:
- net GND: track 336.7 -> 337.4 mm
Changed lines of the file:
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@@
   (via (at 106.55 46.18) (size 0.6858) (drill 0.3302) (layers "F.Cu" "B.Cu") (net 2))
   (via (at 87.87 73.42) (size 0.6858) (drill 0.3302) (layers "F.Cu" "B.Cu") (free) (net 2))
-  (via (at 135.9404 86.684838) (size 0.6858) (drill 0.3302) (layers "F.Cu" "B.Cu") (net 2))
+  (via (at 135.409747 86.249555) (size 0.6858) (drill 0.3302) (layers "F.Cu" "B.Cu") (net 2))
   (via (at 89.37 70.42) (size 0.6858) (drill 0.3302) (layers "F.Cu" "B.Cu") (free) (net 2))
   (via (at 162 56.2) (size 0.6858) (drill 0.3302) (layers "F.Cu" "B.Cu") (net 2))
@@
   (segment (start 168.111638 58.295) (end 167.6727 58.733938) (width 0.25) (layer "B.Cu") (net 2))
   (segment (start 158.128762 64.83) (end 160.3 67.001238) (width 0.508) (layer "B.Cu") (net 2))
+  (segment (start 136.61413 87.453938) (end 137.6577 87.453938) (width 0.254) (layer "B.Cu") (net 2))
   (segment (start 168.4109 51.845) (end 167.6659 51.1) (width 0.508) (layer "B.Cu") (net 2))
   (segment (start 146.86 47.9) (end 146.86 45.335) (width 0.127) (layer "B.Cu") (net 2))
-  (segment (start 136.7095 87.453938) (end 137.6577 87.453938) (width 0.254) (layer "B.Cu") (net 2))
   (segment (start 78.365 70.9) (end 78.415 70.85) (width 0.127) (layer "B.Cu") (net 2))
   (segment (start 117 48.1) (end 116.058762 48.1) (width 0.127) (layer "B.Cu") (net 2))
@@
   (segment (start 108.498636 67.560881) (end 110.649643 67.560881) (width 0.254) (layer "B.Cu") (net 2))
   (segment (start 85.371747 56.023555) (end 85.371747 56.525347) (width 1.016) (layer "B.Cu") (net 2))
-  (segment (start 135.9404 86.684838) (end 136.7095 87.453938) (width 0.254) (layer "B.Cu") (net 2))
   (segment (start 108.498636 68.060881) (end 110.639643 68.060881) (width 0.254) (layer "B.Cu") (net 2))
   (segment (start 145.8597 93.303938) (end 147.0077 94.451938) (width 0.254) (layer "B.Cu") (net 2))
@@
   (segment (start 88.76831 60.143328) (end 88.20828 60.143328) (width 0.127) (layer "B.Cu") (net 2))
   (segment (start 150.4 81.375) (end 150.4 82.675) (width 0.508) (layer "B.Cu") (net 2))
+  (segment (start 135.409747 86.249555) (end 136.61413 87.453938) (width 0.254) (layer "B.Cu") (net 2))
   (segment (start 97.9 82.74) (end 97.9 82.04) (width 0.4) (layer "B.Cu") (net 2))
   (segment (start 91.6927 93.443938) (end 91.668938 93.443938) (width 0.4) (layer "B.Cu") (net 2))
@@
   (via (at 154.915456 68.551764) (size 0.6858) (drill 0.3302) (layers "F.Cu" "B.Cu") (net 99))
   (via (at 143.808191 64.328447) (size 0.6858) (drill 0.3302) (layers "F.Cu" "B.Cu") (net 99))
+  (segment (start 152.68 70.045) (end 153.42222 70.045) (width 0.508) (layer "B.Cu") (net 99))
   (segment (start 161.324062 83.183938) (end 159.216062 83.183938) (width 0.508) (layer "B.Cu") (net 99))
-  (segment (start 152.68 70.045) (end 153.42222 70.045) (width 0.508) (layer "B.Cu") (net 99))
+  (segment (start 162.15 74.635808) (end 162.15 82.358) (width 0.508) (layer "B.Cu") (net 99))
   (segment (start 149.1 63.2) (end 150.5 64.6) (width 0.508) (layer "B.Cu") (net 99))
+  (segment (start 152.68 70.045) (end 152.68 72.73) (width 0.508) (layer "B.Cu") (net 99))
   (segment (start 145.875 63.2) (end 149.1 63.2) (width 0.508) (layer "B.Cu") (net 99))
-  (segment (start 153.15 73.2) (end 160.818762 73.2) (width 0.508) (layer "B.Cu") (net 99))
+  (segment (start 157.55 84.85) (end 157.55 85.175) (width 0.4) (layer "B.Cu") (net 99))
+  (segment (start 159.216062 83.183938) (end 157.55 84.85) (width 0.508) (layer "B.Cu") (net 99))
+  (segment (start 160.714192 73.2) (end 162.15 74.635808) (width 0.508) (layer "B.Cu") (net 99))
   (segment (start 162.15 82.358) (end 161.324062 83.183938) (width 0.508) (layer "B.Cu") (net 99))
-  (segment (start 152.68 70.045) (end 152.68 72.73) (width 0.508) (layer "B.Cu") (net 99))
+  (segment (start 144.625 64.45) (end 145.875 63.2) (width 0.508) (layer "B.Cu") (net 99))
   (segment (start 152.68 72.73) (end 153.15 73.2) (width 0.508) (layer "B.Cu") (net 99))
-  (segment (start 157.55 84.85) (end 157.55 85.175) (width 0.4) (layer "B.Cu") (net 99))
-  (segment (start 162.15 74.531238) (end 162.15 82.358) (width 0.508) (layer "B.Cu") (net 99))
-  (segment (start 144.625 64.45) (end 145.875 63.2) (width 0.508) (layer "B.Cu") (net 99))
   (segment (start 143.929744 64.45) (end 143.808191 64.328447) (width 0.508) (layer "B.Cu") (net 99))
+  (segment (start 153.15 73.2) (end 160.714192 73.2) (width 0.508) (layer "B.Cu") (net 99))
   (segment (start 144.6 64.45) (end 144.625 64.45) (width 0.508) (layer "B.Cu") (net 99))
   (segment (start 153.42222 70.045) (end 154.915456 68.551764) (width 0.508) (layer "B.Cu") (net 99))
-  (segment (start 160.818762 73.2) (end 162.15 74.531238) (width 0.508) (layer "B.Cu") (net 99))
   (segment (start 144.8 64.45) (end 143.929744 64.45) (width 0.508) (layer "B.Cu") (net 99))
-  (segment (start 159.216062 83.183938) (end 157.55 84.85) (width 0.508) (layer "B.Cu") (net 99))
   (segment (start 153 79) (end 154.8 80.8) (width 0.508) (layer "F.Cu") (net 100))
   (segment (start 153 75) (end 153 79) (width 0.508) (layer "F.Cu") (net 100))
